File: pcb/mayavi_ver0.1/mayavi_ver0.1.sch (KiCad schematic (older format))
At the start: 34 parts, among them J3 CONN_01X06, SW1 SW_Push, U2 LIS2DH12, U4 nrf52832, U5 RF_Antenna, Y2 32MHz

Commit message: added schematic
Parts:
- removed U5: RF_Antenna, boostaBLE:Antenna-2.45GHZ_mirror, symbol RF_Antenna
- added AE?: Chip Ant, symbol Antenna
- added C? (x2): 0.1uF, Capacitors_SMD:C_0402, symbol C_Small
- added C?: 2.2pF, boostaBLE:SMD_C0402, symbol C_Small
- added L?: 3.9uH, boostaBLE:SMD_0402, symbol L_Small
- added L?: NC, boostaBLE:SMD_0402, symbol L_Small
- added R?: 100k, symbol R_Small
- added U?: TPS79733MDCKREP, symbol TPS79733MDCKREP
Connections:
- net labels added: BuzN
- net labels removed: BATT_LVL, BLUE, BuzM, GREEN, MODE, P0.26, P0.27, P0.28, P0.29, P0.30, P0.31, RED
- wire segments 182 -> 160
- no-connect marks 17 -> 24
Other:
- note added: "Accelerometer"
- note added: "Power Supply"
- note added: "SWD Programming"
- moved on the sheet: BZ?, J?, R2, R3

Commit message: updated schematic
Parts:
- removed R? (x2): 10K, Resistors_SMD:R_0603, symbol R_Small
- removed SW? (x2): SW_Push, boostaBLE:peter-switch, symbol SW_PUSH
- added R1, R2: 10K, Resistors_SMD:R_0603, symbol R_Small
- added SW1, SW2: SW_Push, boostaBLE:peter-switch, symbol SW_PUSH
- gave numbers to parts that had none: 13
- renumbered C17 to C10, C18 to C11, C19 to C12, C20 to C13, C21 to C15, C22 to C16, C4 to C3, C11 to C6, C12 to C7, C15 to C8, C16 to C9, J3 to J5, L2 to L1, L3 to L2, L4 to L3, R2 to R5, R3 to R6, SW1 to SW3, U4 to U3, Y2 to Y1
Connections:
- net labels removed: 3V3, CS, SDO
- wire segments 160 -> 159
- no-connect marks 24 -> 27
Other:
- moved on the sheet: J4, R5, R6, SW3

Commit message: updated schematic
Parts:
- removed R3: 100k, symbol R_Small
- added R2: 100k, symbol R_Small
- C5: value 0.1uF -> 0.47uF
- renumbered R2 to R3
Connections:
- net VDD: now also R2.1
- net at U1.1 (PG): now also R2.2
Other:
- moved on the sheet: J1

Commit message: updated pcb
Parts:
- removed AE1: Chip Ant, symbol Antenna
- removed C10, C4, C8: 0.1uF, Capacitors_SMD:C_0402, symbol C_Small
- removed C11: 0.8pF, boostaBLE:SMD_C0402, symbol C_Small
- removed C12: 100pF, Capacitors_SMD:C_0402, symbol C_Small
- removed C13: NC, Capacitors_SMD:C_0402, symbol C_Small
- removed C14: 2.2pF, boostaBLE:SMD_C0402, symbol C_Small
- removed C15, C16: 12pF, Capacitors_SMD:C_0402, symbol C_Small
- removed C9: 1uF, Capacitors_SMD:C_0603, symbol C_Small
- removed J4: I2C Test, symbol Conn_01x02
- removed J5: CONN_01X06, Pin_Headers:Pin_Header_Straight_1x06_Pitch2.54mm, symbol CONN_01X06
- removed L1: 15nH, Capacitors_SMD:C_0402, symbol L_Small
- removed L2: 10uH, Inductors_NEOSID:Neosid_Inductor_SM0603CG, symbol L_Small
- removed L3, L5: 3.9uH, boostaBLE:SMD_0402, symbol L_Small
- removed L4: NC, boostaBLE:SMD_0402, symbol L_Small
- removed R2: 100k, symbol R_Small
- removed U1: TPS79733MDCKREP, symbol TPS79733MDCKREP
- removed U3: nrf52832, boostaBLE:nRF52832, symbol nrf52832
- removed Y1: 32MHz, boostaBLE:32MHz_crystal, symbol Crystal_GND24
- added C2: 1uF, Capacitors_SMD:C_0402, symbol C_Small
- added J4: CONN_01X04, Pin_Headers:Pin_Header_Straight_1x04_Pitch1.27mm, symbol CONN_01X04
- added L1, L2: 10uH, Inductors_SMD:L_0603, symbol L
- added U1: MCP1702, TO_SOT_Packages_SMD:SOT-23, symbol MCP1700-1202E_SOT23
- added U3: MDBT42V, mayavi:MDBT42V, symbol MDBT42V
- BZ1: footprint (none) -> mayavi:PKMCS0909E4000-R1
- C5: value 0.47uF -> 10uF
- C6: value 0.1uF -> 10uF
- C7: value 4.7uF -> 1uF; footprint Capacitors_SMD:C_0603 -> Capacitors_SMD:C_0402
- J1, J2: footprint (none) -> Pin_Headers:Pin_Header_Straight_1x02_Pitch2.54mm
- J3: footprint (none) -> Pin_Headers:Pin_Header_Straight_1x04_Pitch2.54mm
- SW1, SW2, SW3: footprint boostaBLE:peter-switch -> mayavi:peter-switch
- U2: footprint boostaBLE:LIS2DH12-LGA12_2X2MM -> mayavi:LIS2DH12-LGA12_2X2MM
- renumbered C2 to C3, C3 to C4, R3 to R2, R4 to R3, R5 to R4, R6 to R5
Connections:
- net BuzN: now also U3.12 (P0.08)
- net BuzP: now also U3.11 (P0.09)
- net GND: now also C2.2, J4.4 (P4), U1.1 (GND), U3.1 (GND), U3.10 (GND), U3.18 (GND), U3.29 (GND)
- net INT1: now also U3.26 (P0.02)
- net INT2: now also U3.25 (P0.25)
- net RESET: now also U3.3 (RESET/P0.21); no longer R2.2, R3.2, SW2.1, SW3.1
- net SCL: now also U3.28 (P0.11)
- net SDA: now also U3.27 (P0.03)
- net SWDCLK: now also J4.2 (P2), U3.2 (SWDCLK)
- net SWDIO: now also J4.1 (P1), U3.4 (SWDIO)
- net VBAT: now also C2.1, U1.3 (VI)
- net VDD: now also C6.1, J4.3 (P3), U1.2 (VO), U3.20 (VCC); no longer C7.1
- new net: C7.1, L2.2, U3.21 (DEC4)
- new net: L1.1, U3.22 (DCC)
- new net: L1.2, L2.1
- new net BTN1: R2.2, SW2.1, U3.14 (P0.06)
- new net BTN2: R3.2, SW3.1, U3.13 (P0.10)
- no-connect marks 27 -> 12
Other:
- note added: "Buttons"
- note added: "I2C Pull-ups"
- moved on the sheet: BZ1, C1, C3, C4, J1, J2, J3, R1, R2, R3, R4, R5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

Commit message: updated pcb
Parts:
- removed R1: 10K, Resistors_SMD:R_0603, symbol R_Small
- removed SW1: SW_Push, mayavi:peter-switch, symbol SW_PUSH
- J1: footprint Pin_Headers:Pin_Header_Straight_1x02_Pitch2.54mm -> Pin_Headers:Pin_Header_Straight_1x02_Pitch1.27mm
- J2: footprint Pin_Headers:Pin_Header_Straight_1x02_Pitch2.54mm -> Pin_Headers:Pin_Header_Angled_1x02_Pitch2.54mm
- J4: value CONN_01X04 -> SWD header; footprint Pin_Headers:Pin_Header_Straight_1x04_Pitch1.27mm -> mayavi:SWD_1.27
- SW1: renamed from SW2; footprint mayavi:peter-switch -> mayavi:SW5052
- SW2: renamed from SW3; footprint mayavi:peter-switch -> mayavi:SW5052
- renumbered R2 to R1, R3 to R2, R4 to R3, R5 to R4
Connections:
- net RESET: no longer names the net of U3.3 (RESET/P0.21)
- no-connect marks 12 -> 13
Changed lines of the file:
@@
 LIBS:valves
 LIBS:mayavi
-LIBS:bluestone_tracker_ Lipo
-LIBS:bluestone_tracker
 LIBS:mayavi_ver0.1-cache
 EELAYER 25 0
@@
 $EndComp
 $Comp
-L R_Small R4
+L R_Small R3
 U 1 1 5A2BED80
 P 8420 5785
-F 0 "R4" H 8450 5805 50  0000 L CNN
+F 0 "R3" H 8450 5805 50  0000 L CNN
 F 1 "10K" H 8450 5745 50  0000 L CNN
 F 2 "Resistors_SMD:R_0603" H 8420 5785 50  0001 C CNN
@@
 $EndComp
 $Comp
-L R_Small R5
+L R_Small R4
 U 1 1 5A2BEF53
 P 8550 5785
-F 0 "R5" H 8580 5805 50  0000 L CNN
+F 0 "R4" H 8580 5805 50  0000 L CNN
 F 1 "10K" H 8580 5745 50  0000 L CNN
 F 2 "Resistors_SMD:R_0603" H 8550 5785 50  0001 C CNN
@@
 INT2
 $Comp
-L SW_PUSH SW3
+L SW_PUSH SW2
 U 1 1 5A2BB78D
 P 6365 6105
-F 0 "SW3" H 6415 6205 50  0000 L CNN
+F 0 "SW2" H 6415 6205 50  0000 L CNN
 F 1 "SW_Push" H 6365 6045 50  0000 C CNN
-F 2 "mayavi:peter-switch" H 6365 6305 50  0001 C CNN
+F 2 "mayavi:SW5052" H 6365 6305 50  0001 C CNN
 F 3 "" H 6365 6305 50  0001 C CNN
 	1    6365 6105
@@
 $EndComp
 $Comp
-L R_Small R3
+L R_Small R2
 U 1 1 5A2BDA80
 P 6365 5490
-F 0 "R3" H 6395 5510 50  0000 L CNN
+F 0 "R2" H 6395 5510 50  0000 L CNN
 F 1 "10K" H 6395 5450 50  0000 L CNN
 F 2 "Resistors_SMD:R_0603" H 6365 5490 50  0001 C CNN
@@
 F 0 "J2" H 5940 2835 50  0000 C CNN
 F 1 "Charging Conn" H 5940 2535 50  0000 C CNN
-F 2 "Pin_Headers:Pin_Header_Straight_1x02_Pitch2.54mm" H 5940 2735 50  0001 C CNN
+F 2 "Pin_Headers:Pin_Header_Angled_1x02_Pitch2.54mm" H 5940 2735 50  0001 C CNN
 F 3 "" H 5940 2735 50  0001 C CNN
 	1    5940 2735
@@
 F 0 "J1" H 3780 3895 50  0000 C CNN
 F 1 "3.7V LiPo" H 3780 3595 50  0000 C CNN
-F 2 "Pin_Headers:Pin_Header_Straight_1x02_Pitch2.54mm" H 3780 3795 50  0001 C CNN
+F 2 "Pin_Headers:Pin_Header_Straight_1x02_Pitch1.27mm" H 3780 3795 50  0001 C CNN
 F 3 "" H 3780 3795 50  0001 C CNN
 	1    3780 3795
@@
 Power Supply
 $Comp
-L SW_PUSH SW2
+L SW_PUSH SW1
 U 1 1 5B23DC27
 P 5285 6110
-F 0 "SW2" H 5335 6210 50  0000 L CNN
+F 0 "SW1" H 5335 6210 50  0000 L CNN
 F 1 "SW_Push" H 5285 6050 50  0000 C CNN
-F 2 "mayavi:peter-switch" H 5285 6310 50  0001 C CNN
+F 2 "mayavi:SW5052" H 5285 6310 50  0001 C CNN
 F 3 "" H 5285 6310 50  0001 C CNN
 	1    5285 6110
@@
 $EndComp
 $Comp
-L R_Small R2
+L R_Small R1
 U 1 1 5B23DC33
 P 5285 5495
-F 0 "R2" H 5315 5515 50  0000 L CNN
+F 0 "R1" H 5315 5515 50  0000 L CNN
 F 1 "10K" H 5315 5455 50  0000 L CNN
 F 2 "Resistors_SMD:R_0603" H 5285 5495 50  0001 C CNN
@@
 BTN1
 $Comp
-L SW_PUSH SW1
-U 1 1 5B23DCDB
-P 4070 6110
-F 0 "SW1" H 4120 6210 50  0000 L CNN
-F 1 "SW_Push" H 4070 6050 50  0000 C CNN
-F 2 "mayavi:peter-switch" H 4070 6310 50  0001 C CNN
-F 3 "" H 4070 6310 50  0001 C CNN
-	1    4070 6110
-	0    1    1    0
-$EndComp
-$Comp
-L GND #PWR012
-U 1 1 5B23DCE1
-P 4070 6470
-F 0 "#PWR012" H 4070 6220 50  0001 C CNN
-F 1 "GND" H 4070 6320 50  0000 C CNN
-F 2 "" H 4070 6470 50  0001 C CNN
-F 3 "" H 4070 6470 50  0001 C CNN
-	1    4070 6470
-	1    0    0    -1
-$EndComp
-$Comp
-L R_Small R1
-U 1 1 5B23DCE7
-P 4070 5495
-F 0 "R1" H 4100 5515 50  0000 L CNN
-F 1 "10K" H 4100 5455 50  0000 L CNN
-F 2 "Resistors_SMD:R_0603" H 4070 5495 50  0001 C CNN
-F 3 "" H 4070 5495 50  0001 C CNN
-	1    4070 5495
-	1    0    0    -1
-$EndComp
-Text GLabel 3755 5295 0    39   Input ~ 0
-VDD
-Text GLabel 3755 5710 0    39   Input ~ 0
-RESET
-$Comp
-L PWR_FLAG #FLG013
+L PWR_FLAG #FLG012
 U 1 1 5B23FF84
 P 3345 3080
-F 0 "#FLG013" H 3345 3155 50  0001 C CNN
+F 0 "#FLG012" H 3345 3155 50  0001 C CNN
 F 1 "PWR_FLAG" H 3345 3230 50  0000 C CNN
 F 2 "" H 3345 3080 50  0001 C CNN
@@
 $EndComp
 $Comp
-L GND #PWR014
+L GND #PWR013
 U 1 1 5B240BD3
 P 3345 3115
-F 0 "#PWR014" H 3345 2865 50  0001 C CNN
+F 0 "#PWR013" H 3345 2865 50  0001 C CNN
 F 1 "GND" H 3345 2965 50  0000 C CNN
 F 2 "" H 3345 3115 50  0001 C CNN
@@
 $EndComp
 $Comp
-L PWR_FLAG #FLG015
+L PWR_FLAG #FLG014
 U 1 1 5B2408BF
 P 3365 2570
-F 0 "#FLG015" H 3365 2645 50  0001 C CNN
+F 0 "#FLG014" H 3365 2645 50  0001 C CNN
 F 1 "PWR_FLAG" H 3365 2720 50  0000 C CNN
 F 2 "" H 3365 2570 50  0001 C CNN
@@
 $EndComp
 $Comp
-L GND #PWR016
+L GND #PWR015
 U 1 1 5B35B4C1
 P 10555 4295
-F 0 "#PWR016" H 10555 4045 50  0001 C CNN
+F 0 "#PWR015" H 10555 4045 50  0001 C CNN
 F 1 "GND" H 10555 4145 50  0000 C CNN
 F 2 "" H 10555 4295 50  0001 C CNN
@@
 $EndComp
 $Comp
-L GND #PWR017
+L GND #PWR016
 U 1 1 5B35B98A
 P 11045 2815
-F 0 "#PWR017" H 11045 2565 50  0001 C CNN
+F 0 "#PWR016" H 11045 2565 50  0001 C CNN
 F 1 "GND" H 11045 2665 50  0000 C CNN
 F 2 "" H 11045 2815 50  0001 C CNN
@@
 $EndComp
 $Comp
-L GND #PWR018
+L GND #PWR017
 U 1 1 5B35CA9F
 P 12425 4520
-F 0 "#PWR018" H 12425 4270 50  0001 C CNN
+F 0 "#PWR017" H 12425 4270 50  0001 C CNN
 F 1 "GND" H 12425 4370 50  0000 C CNN
 F 2 "" H 12425 4520 50  0001 C CNN
@@
 $EndComp
 $Comp
-L GND #PWR019
+L GND #PWR018
 U 1 1 5B35CAFB
 P 12685 2780
-F 0 "#PWR019" H 12685 2530 50  0001 C CNN
+F 0 "#PWR018" H 12685 2530 50  0001 C CNN
 F 1 "GND" H 12685 2630 50  0000 C CNN
 F 2 "" H 12685 2780 50  0001 C CNN
@@
 $EndComp
 $Comp
-L GND #PWR020
+L GND #PWR019
 U 1 1 5B35F6A7
 P 10970 4925
-F 0 "#PWR020" H 10970 4675 50  0001 C CNN
+F 0 "#PWR019" H 10970 4675 50  0001 C CNN
 F 1 "GND" H 10970 4775 50  0000 C CNN
 F 2 "" H 10970 4925 50  0001 C CNN
@@
 $EndComp
 $Comp
-L GND #PWR021
+L GND #PWR020
 U 1 1 5B35FA52
 P 10975 5325
-F 0 "#PWR021" H 10975 5075 50  0001 C CNN
+F 0 "#PWR020" H 10975 5075 50  0001 C CNN
 F 1 "GND" H 10975 5175 50  0000 C CNN
 F 2 "" H 10975 5325 50  0001 C CNN
@@
 P 11395 7185
 F 0 "J4" H 11395 7435 50  0000 C CNN
-F 1 "CONN_01X04" V 11495 7185 50  0000 C CNN
-F 2 "Pin_Headers:Pin_Header_Straight_1x04_Pitch1.27mm" H 11395 7185 50  0001 C CNN
+F 1 "SWD header" V 11495 7185 50  0000 C CNN
+F 2 "mayavi:SWD_1.27" H 11395 7185 50  0001 C CNN
 F 3 "" H 11395 7185 50  0001 C CNN
 	1    11395 7185
@@
 Text GLabel 12325 5100 2    39   Input ~ 0
 INT2
-Text GLabel 12410 2480 2    39   Input ~ 0
-RESET
 NoConn ~ 11785 2865
 NoConn ~ 11885 2865
@@
 	3345 3080 3345 3115
 Wire Wire Line
-	4070 6410 4070 6470
-Connection ~ 4070 5710
-Wire Wire Line
-	3755 5710 4070 5710
-Wire Wire Line
-	4070 5595 4070 5810
-Wire Wire Line
-	4070 5295 3755 5295
-Wire Wire Line
-	4070 5395 4070 5295
-Wire Wire Line
 	5285 6410 5285 6470
 Connection ~ 5285 5710
@@
 	6450 8010 6270 8010
 Wire Wire Line
-	12180 2480 12410 2480
-Wire Wire Line
-	12180 2480 12180 2865
-Wire Wire Line
 	12410 2380 12080 2375
 Wire Wire Line
@@
 Wire Wire Line
 	6175 4060 6175 3995
+NoConn ~ 12180 2865
 $EndSCHEMATC
